Commit message: add a gripper urdf

File: src/my_robot_description/urdf/mtl.urdf.xacro (robot description, xacro)
@@ -19,3 +19,9 @@
         <color rgba="0.0 0.0 0.0 1" />
     </material>
+    <material name="dark_red">
+        <color rgba="0.4 0 0 0.8" />
+    </material>
+    <material name="dark_green">
+        <color rgba="0.0 0.4 0 0.8" />
+    </material>
 </robot>
