Commit message: attach the gripper to tool_link

File: src/my_robot_description/urdf/gripper.urdf.xacro (robot description, xacro)
@@ -1,4 +1,4 @@
 <?xml version="1.0"?>
-<robot name="gripper" xmlns:xacro="http://www.ros.org/wiki/xacro">
+<robot xmlns:xacro="http://www.ros.org/wiki/xacro">
     <link name="gripper_base_link">
         <visual>

File: src/my_robot_description/urdf/robot.urdf.xacro (robot description, xacro)
@@ -3,3 +3,10 @@
     <xacro:include filename="mtl.urdf.xacro" />
     <xacro:include filename="arm.urdf.xacro" />
+    <xacro:include filename="gripper.urdf.xacro" />
+    <!-- Connect the gripper to ef -->
+    <joint name="gripper_base_joint" type="fixed">
+        <parent link="tool_link" />
+        <child link="gripper_base_link" />
+        <origin xyz="0 0 0" rpy="0 0 0" />
+    </joint>
 </robot>
