Commit message: refactor the URDF

File: src/my_robot_description/urdf/arm.urdf.xacro (robot description, xacro)
@@ -1,5 +1,4 @@
 <?xml version="1.0"?>
-<robot name="my_arm" xmlns:xacro="http://www.ros.org/wiki/xacro">
-    <xacro:include filename="mtl.urdf.xacro" />
+<robot xmlns:xacro="http://www.ros.org/wiki/xacro">
     <!-- Base Link-->
     <link name="base_link">
@@ -9,5 +8,5 @@
             </geometry>
             <origin xyz="0 0 0.05" rpy="0 0 0" />
-            <material name="grey" />
+            <material name="black" />
         </visual>
     </link>
@@ -53,5 +52,5 @@
             </geometry>
             <origin xyz="0 0 0.05" rpy="0 0 0" />
-            <material name="blue" />
+            <material name="orange" />
         </visual>
     </link>
@@ -70,5 +69,5 @@
             </geometry>
             <origin xyz="0 0 0.25" rpy="0 0 0" />
-            <material name="grey" />
+            <material name="white" />
         </visual>
     </link>
@@ -87,5 +86,5 @@
             </geometry>
             <origin xyz="0 0 0.025" rpy="0 0 0" />
-            <material name="blue" />
+            <material name="yellow" />
         </visual>
     </link>

File: src/my_robot_description/urdf/mtl.urdf.xacro (robot description, xacro)
@@ -13,3 +13,9 @@
         <color rgba="1.0 1.0 0 1" />
     </material>
+    <material name="white">
+        <color rgba="1.0 1.0 1.0 1" />
+    </material>
+    <material name="black">
+        <color rgba="0.0 0.0 0.0 1" />
+    </material>
 </robot>

Commit message: add collision tags

File: src/my_robot_description/urdf/arm.urdf.xacro (robot description, xacro)
@@ -10,4 +10,10 @@
             <material name="black" />
         </visual>
+        <collision>
+            <geometry>
+                <box size="0.4 0.4 0.1" />
+            </geometry>
+            <origin xyz="0 0 0.05" rpy="0 0 0" />
+        </collision>
     </link>
     <!-- Shoulder link -->
@@ -20,4 +26,10 @@
             <material name="blue" />
         </visual>
+        <collision>
+            <geometry>
+                <box size="0.2 0.2 0.5" />
+            </geometry>
+            <origin xyz="0 0 0.25" rpy="0 0 0" />
+        </collision>
     </link>
     <joint name="joint1" type="revolute">
@@ -37,4 +49,10 @@
             <material name="grey" />
         </visual>
+        <collision>
+            <geometry>
+                <box size="0.1 0.1 0.6" />
+            </geometry>
+            <origin xyz="0 0 0.3" rpy="0 0 0" />
+        </collision>
     </link>
     <joint name="joint2" type="revolute">
@@ -54,4 +72,10 @@
             <material name="orange" />
         </visual>
+        <collision>
+            <geometry>
+                <box size="0.1 0.1 0.1" />
+            </geometry>
+            <origin xyz="0 0 0.05" rpy="0 0 0" />
+        </collision>
     </link>
     <joint name="joint3" type="revolute">
@@ -71,4 +95,10 @@
             <material name="white" />
         </visual>
+        <collision>
+            <geometry>
+                <box size="0.1 0.1 0.5" />
+            </geometry>
+            <origin xyz="0 0 0.25" rpy="0 0 0" />
+        </collision>
     </link>
     <joint name="joint4" type="revolute">
@@ -88,4 +118,10 @@
             <material name="yellow" />
         </visual>
+        <collision>
+            <geometry>
+                <box size="0.1 0.1 0.05" />
+            </geometry>
+            <origin xyz="0 0 0.025" rpy="0 0 0" />
+        </collision>
     </link>
     <joint name="joint5" type="revolute">
@@ -105,4 +141,10 @@
             <material name="grey" />
         </visual>
+        <collision>
+            <geometry>
+                <box size="0.1 0.1 0.02" />
+            </geometry>
+            <origin xyz="0 0 0.01" rpy="0 0 0" />
+        </collision>
     </link>
     <joint name="joint6" type="continuous">

Commit message: add a mobile base and assemble the arm on top

File: src/my_robot_description/urdf/arm.urdf.xacro (robot description, xacro)
@@ -2,5 +2,5 @@
 <robot xmlns:xacro="http://www.ros.org/wiki/xacro">
     <!-- Base Link-->
-    <link name="base_link">
+    <link name="arm_base_link">
         <visual>
             <geometry>
@@ -34,5 +34,5 @@
     </link>
     <joint name="joint1" type="revolute">
-        <parent link="base_link" />
+        <parent link="arm_base_link" />
         <child link="shoulder_link" />
         <origin xyz="0 0 0.1" rpy="0 0 0" />

File: src/my_robot_moveit_config/config/my_arm.urdf.xacro (robot description, xacro)
@@ -3,7 +3,8 @@
     <xacro:arg name="initial_positions_file" default="initial_positions.yaml" />
     <!-- Import my_arm urdf file -->
-    <xacro:include filename="$(find my_robot_description)/urdf/robot.urdf.xacro" />
+    <xacro:include filename="$(find my_robot_description)/urdf/arm_with_gripper.urdf.xacro" />
     <!-- Import control_xacro -->
     <xacro:include filename="my_arm.ros2_control.xacro" />
-    <xacro:my_arm_ros2_control name="FakeSystem" initial_positions_file="$(arg initial_positions_file)"/>
+    <xacro:my_arm_ros2_control name="FakeSystem"
+        initial_positions_file="$(arg initial_positions_file)" />
 </robot>
