Commit message: rename the arm package to arm_movit

File: src/my_robot_description/urdf/platform.xacro (robot description, xacro)
@@ -5,7 +5,4 @@
     <xacro:include filename="gripper.urdf.xacro" />
     <xacro:include filename="mobile_base.urdf.xacro" />
-    <xacro:include filename="ros2_control/mobile_base.ros2_control.xacro" />
-    <xacro:include filename="ros2_control/arm.ros2_control.xacro" />
-    <xacro:include filename="ros2_control/gripper.ros2_control.xacro" />
     <!-- Connect the gripper to ef -->
     <joint name="gripper_base_joint" type="fixed">
@@ -17,5 +14,5 @@
     <joint name="arm_base_joint" type="fixed">
         <parent link="mobile_base_link" />
-        <child link="base_link" />
+        <child link="arm_base_link" />
         <origin xyz="0 0 0.3" rpy="0 0 0" />
     </joint>
