Commit message: update movit for the gripper

File: src/my_robot_moveit_config/config/my_arm.ros2_control.xacro (robot description, xacro)
@@ -50,4 +50,11 @@
                 <state_interface name="velocity"/>
             </joint>
+            <joint name="gripper_left_finger_joint">
+                <command_interface name="position"/>
+                <state_interface name="position">
+                  <param name="initial_value">${initial_positions['gripper_left_finger_joint']}</param>
+                </state_interface>
+                <state_interface name="velocity"/>
+            </joint>
         </ros2_control>
     </xacro:macro>
